Commit message: Add reacher real world script for FR3

File: content/assets/urdf/franka_description/franka_panda_no_gripper.urdf (robot description, URDF)
Before this commit: robot panda, 11 links, 10 joints
Joints:
- joint panda_joint1: limit lower=-2.8973 upper=2.8973 effort=87 velocity=2.1750 -> lower=-2.3093 upper=2.3093 effort=87 velocity=2.0
- joint panda_joint2: limit lower=-1.7628 upper=1.7628 effort=87 velocity=2.1750 -> lower=-1.5133 upper=1.5133 effort=87 velocity=1.0
- joint panda_joint3: limit lower=-2.8973 upper=2.8973 effort=87 velocity=2.1750 -> lower=-2.4937 upper=2.4937 effort=87 velocity=1.50
- joint panda_joint4: limit lower=-3.0718 upper=-0.0698 effort=87 velocity=2.1750 -> lower=-2.7478 upper=-0.4461 effort=87 velocity=1.25
- joint panda_joint5: limit lower=-2.8973 upper=2.8973 effort=12 velocity=2.6100 -> lower=-2.4800 upper=2.4800 effort=12 velocity=3.00
- joint panda_joint6: limit lower=-0.0175 upper=3.7525 effort=12 velocity=2.6100 -> lower=0.8521 upper=4.2094 effort=12 velocity=1.50
- joint panda_joint7: limit lower=-2.8973 upper=2.8973 effort=12 velocity=2.6100 -> lower=-2.6895 upper=2.6895 effort=12 velocity=3.00
